Commit message: updated gazebo_wheel.launch

File: quadruped_description/xacros/gazebo_plugin.xacro (robot description, xacro)
@@ -1,4 +1,4 @@
 <?xml version="1.0"?>
-<robot name="quad_wheel" xmlns:xacro="http://www.ros.org/wiki/xacro">
+<robot name="quadruped" xmlns:xacro="http://www.ros.org/wiki/xacro">
     <xacro:macro name="gazebo_plugin">
         <!-- Enable the Joint Control -->

File: quadruped_description/xacros/material.xacro (robot description, xacro)
@@ -1,4 +1,4 @@
 <?xml version="1.0"?>
-<robot name="quad_wheel" xmlns:xacro="http://www.ros.org/wiki/xacro">
+<robot name="quadruped" xmlns:xacro="http://www.ros.org/wiki/xacro">
     <xacro:macro name="material" params="name color0 color1 color2 color3 colorw">
         <gazebo reference="${name}_link_0">

File: quadruped_description/xacros/quad_wheel.xacro (robot description, xacro)
@@ -1,5 +1,5 @@
 <?xml version="1.0"?>
-<robot name="quad_wheel" xmlns:xacro="http://wiki.ros.org/xacro">
- <xacro:macro name="qhumus_b">
+<robot name="quadruped" xmlns:xacro="http://wiki.ros.org/xacro">
+ <xacro:macro name="quadruped">
   <link
     name="base_link">
@@ -24,19 +24,19 @@
       <geometry>
         <mesh
-          filename="package://quadruped_with_wheel_urdf/meshes/base_link.STL" />
-      </geometry>
-      <material
-        name="">
-        <color
-          rgba="0.792156862745098 0.819607843137255 0.933333333333333 1" />
-      </material>
-    </visual>
-    <collision>
-      <origin
-        xyz="0 0 0"
-        rpy="0 0 0" />
-      <geometry>
-        <mesh
-          filename="package://quadruped_with_wheel_urdf/meshes/base_link.STL" />
+          filename="package://quadruped_description/meshes/base_link.STL" />
+      </geometry>
+      <material
+        name="">
+        <color
+          rgba="0.792156862745098 0.819607843137255 0.933333333333333 1" />
+      </material>
+    </visual>
+    <collision>
+      <origin
+        xyz="0 0 0"
+        rpy="0 0 0" />
+      <geometry>
+        <mesh
+          filename="package://quadruped_description/meshes/base_link.STL" />
       </geometry>
     </collision>
@@ -64,19 +64,19 @@
       <geometry>
         <mesh
-          filename="package://quadruped_with_wheel_urdf/meshes/L1_link_0.STL" />
-      </geometry>
-      <material
-        name="">
-        <color
-          rgba="0.792156862745098 0.819607843137255 0.933333333333333 1" />
-      </material>
-    </visual>
-    <collision>
-      <origin
-        xyz="0 0 0"
-        rpy="0 0 0" />
-      <geometry>
-        <mesh
-          filename="package://quadruped_with_wheel_urdf/meshes/L1_link_0.STL" />
+          filename="package://quadruped_description/meshes/L1_link_0.STL" />
+      </geometry>
+      <material
+        name="">
+        <color
+          rgba="0.792156862745098 0.819607843137255 0.933333333333333 1" />
+      </material>
+    </visual>
+    <collision>
+      <origin
+        xyz="0 0 0"
+        rpy="0 0 0" />
+      <geometry>
+        <mesh
+          filename="package://quadruped_description/meshes/L1_link_0.STL" />
       </geometry>
     </collision>
@@ -117,19 +117,19 @@
       <geometry>
         <mesh
-          filename="package://quadruped_with_wheel_urdf/meshes/L1_link_1.STL" />
-      </geometry>
-      <material
-        name="">
-        <color
-          rgba="0.792156862745098 0.819607843137255 0.933333333333333 1" />
-      </material>
-    </visual>
-    <collision>
-      <origin
-        xyz="0 0 0"
-        rpy="0 0 0" />
-      <geometry>
-        <mesh
-          filename="package://quadruped_with_wheel_urdf/meshes/L1_link_1.STL" />
+          filename="package://quadruped_description/meshes/L1_link_1.STL" />
+      </geometry>
+      <material
+        name="">
+        <color
+          rgba="0.792156862745098 0.819607843137255 0.933333333333333 1" />
+      </material>
+    </visual>
+    <collision>
+      <origin
+        xyz="0 0 0"
+        rpy="0 0 0" />
+      <geometry>
+        <mesh
+          filename="package://quadruped_description/meshes/L1_link_1.STL" />
       </geometry>
     </collision>
@@ -175,19 +175,19 @@
       <geometry>
         <mesh
-          filename="package://quadruped_with_wheel_urdf/meshes/L1_link_2.STL" />
-      </geometry>
-      <material
-        name="">
-        <color
-          rgba="0.792156862745098 0.819607843137255 0.933333333333333 1" />
-      </material>
-    </visual>
-    <collision>
-      <origin
-        xyz="0 0 0"
-        rpy="0 0 0" />
-      <geometry>
-        <mesh
-          filename="package://quadruped_with_wheel_urdf/meshes/L1_link_2.STL" />
+          filename="package://quadruped_description/meshes/L1_link_2.STL" />
+      </geometry>
+      <material
+        name="">
+        <color
+          rgba="0.792156862745098 0.819607843137255 0.933333333333333 1" />
+      </material>
+    </visual>
+    <collision>
+      <origin
+        xyz="0 0 0"
+        rpy="0 0 0" />
+      <geometry>
+        <mesh
+          filename="package://quadruped_description/meshes/L1_link_2.STL" />
       </geometry>
     </collision>
@@ -233,19 +233,19 @@
       <geometry>
         <mesh
-          filename="package://quadruped_with_wheel_urdf/meshes/L1_link_3.STL" />
-      </geometry>
-      <material
-        name="">
-        <color
-          rgba="0.792156862745098 0.819607843137255 0.933333333333333 1" />
-      </material>
-    </visual>
-    <collision>
-      <origin
-        xyz="0 0 0"
-        rpy="0 0 0" />
-      <geometry>
-        <mesh
-          filename="package://quadruped_with_wheel_urdf/meshes/L1_link_3.STL" />
+          filename="package://quadruped_description/meshes/L1_link_3.STL" />
+      </geometry>
+      <material
+        name="">
+        <color
+          rgba="0.792156862745098 0.819607843137255 0.933333333333333 1" />
+      </material>
+    </visual>
+    <collision>
+      <origin
+        xyz="0 0 0"
+        rpy="0 0 0" />
+      <geometry>
+        <mesh
+          filename="package://quadruped_description/meshes/L1_link_3.STL" />
       </geometry>
     </collision>
@@ -291,5 +291,5 @@
       <geometry>
         <mesh
-          filename="package://quadruped_with_wheel_urdf/meshes/L1_w.STL" />
+          filename="package://quadruped_description/meshes/L1_w.STL" />
       </geometry>
       <material
@@ -305,5 +305,5 @@
       <geometry>
         <mesh
-          filename="package://quadruped_with_wheel_urdf/meshes/L1_w.STL" />
+          filename="package://quadruped_description/meshes/L1_w.STL" />
       </geometry>
     </collision>
@@ -349,19 +349,19 @@
       <geometry>
         <mesh
-          filename="package://quadruped_with_wheel_urdf/meshes/L2_link_0.STL" />
-      </geometry>
-      <material
-        name="">
-        <color
-          rgba="0.792156862745098 0.819607843137255 0.933333333333333 1" />
-      </material>
-    </visual>
-    <collision>
-      <origin
-        xyz="0 0 0"
-        rpy="0 0 0" />
-      <geometry>
-        <mesh
-          filename="package://quadruped_with_wheel_urdf/meshes/L2_link_0.STL" />
+          filename="package://quadruped_description/meshes/L2_link_0.STL" />
+      </geometry>
+      <material
+        name="">
+        <color
+          rgba="0.792156862745098 0.819607843137255 0.933333333333333 1" />
+      </material>
+    </visual>
+    <collision>
+      <origin
+        xyz="0 0 0"
+        rpy="0 0 0" />
+      <geometry>
+        <mesh
+          filename="package://quadruped_description/meshes/L2_link_0.STL" />
       </geometry>
     </collision>
@@ -402,19 +402,19 @@
       <geometry>
         <mesh
-          filename="package://quadruped_with_wheel_urdf/meshes/L2_link_1.STL" />
-      </geometry>
-      <material
-        name="">
-        <color
-          rgba="0.792156862745098 0.819607843137255 0.933333333333333 1" />
-      </material>
-    </visual>
-    <collision>
-      <origin
-        xyz="0 0 0"
-        rpy="0 0 0" />
-      <geometry>
-        <mesh
-          filename="package://quadruped_with_wheel_urdf/meshes/L2_link_1.STL" />
+          filename="package://quadruped_description/meshes/L2_link_1.STL" />
+      </geometry>
+      <material
+        name="">
+        <color
+          rgba="0.792156862745098 0.819607843137255 0.933333333333333 1" />
+      </material>
+    </visual>
+    <collision>
+      <origin
+        xyz="0 0 0"
+        rpy="0 0 0" />
+      <geometry>
+        <mesh
+          filename="package://quadruped_description/meshes/L2_link_1.STL" />
       </geometry>
     </collision>
@@ -460,19 +460,19 @@
       <geometry>
         <mesh
-          filename="package://quadruped_with_wheel_urdf/meshes/L2_link_2.STL" />
-      </geometry>
-      <material
-        name="">
-        <color
-          rgba="0.792156862745098 0.819607843137255 0.933333333333333 1" />
-      </material>
-    </visual>
-    <collision>
-      <origin
-        xyz="0 0 0"
-        rpy="0 0 0" />
-      <geometry>
-        <mesh
-          filename="package://quadruped_with_wheel_urdf/meshes/L2_link_2.STL" />
+          filename="package://quadruped_description/meshes/L2_link_2.STL" />
+      </geometry>
+      <material
+        name="">
+        <color
+          rgba="0.792156862745098 0.819607843137255 0.933333333333333 1" />
+      </material>
+    </visual>
+    <collision>
+      <origin
+        xyz="0 0 0"
+        rpy="0 0 0" />
+      <geometry>
+        <mesh
+          filename="package://quadruped_description/meshes/L2_link_2.STL" />
       </geometry>
     </collision>
@@ -518,19 +518,19 @@
       <geometry>
         <mesh
-          filename="package://quadruped_with_wheel_urdf/meshes/L2_link_3.STL" />
-      </geometry>
-      <material
-        name="">
-        <color
-          rgba="0.792156862745098 0.819607843137255 0.933333333333333 1" />
-      </material>
-    </visual>
-    <collision>
-      <origin
-        xyz="0 0 0"
-        rpy="0 0 0" />
-      <geometry>
-        <mesh
-          filename="package://quadruped_with_wheel_urdf/meshes/L2_link_3.STL" />
+          filename="package://quadruped_description/meshes/L2_link_3.STL" />
+      </geometry>
+      <material
+        name="">
+        <color
+          rgba="0.792156862745098 0.819607843137255 0.933333333333333 1" />
+      </material>
+    </visual>
+    <collision>
+      <origin
+        xyz="0 0 0"
+        rpy="0 0 0" />
+      <geometry>
+        <mesh
+          filename="package://quadruped_description/meshes/L2_link_3.STL" />
       </geometry>
     </collision>
@@ -576,5 +576,5 @@
       <geometry>
         <mesh
-          filename="package://quadruped_with_wheel_urdf/meshes/L2_w.STL" />
+          filename="package://quadruped_description/meshes/L2_w.STL" />
       </geometry>
       <material
@@ -590,5 +590,5 @@
       <geometry>
         <mesh
-          filename="package://quadruped_with_wheel_urdf/meshes/L2_w.STL" />
+          filename="package://quadruped_description/meshes/L2_w.STL" />
       </geometry>
     </collision>
@@ -634,19 +634,19 @@
       <geometry>
         <mesh
-          filename="package://quadruped_with_wheel_urdf/meshes/L3_link_0.STL" />
-      </geometry>
-      <material
-        name="">
-        <color
-          rgba="0.792156862745098 0.819607843137255 0.933333333333333 1" />
-      </material>
-    </visual>
-    <collision>
-      <origin
-        xyz="0 0 0"
-        rpy="0 0 0" />
-      <geometry>
-        <mesh
-          filename="package://quadruped_with_wheel_urdf/meshes/L3_link_0.STL" />
+          filename="package://quadruped_description/meshes/L3_link_0.STL" />
+      </geometry>
+      <material
+        name="">
+        <color
+          rgba="0.792156862745098 0.819607843137255 0.933333333333333 1" />
+      </material>
+    </visual>
+    <collision>
+      <origin
+        xyz="0 0 0"
+        rpy="0 0 0" />
+      <geometry>
+        <mesh
+          filename="package://quadruped_description/meshes/L3_link_0.STL" />
       </geometry>
     </collision>
@@ -687,19 +687,19 @@
       <geometry>
         <mesh
-          filename="package://quadruped_with_wheel_urdf/meshes/L3_Link_1.STL" />
-      </geometry>
-      <material
-        name="">
-        <color
-          rgba="0.792156862745098 0.819607843137255 0.933333333333333 1" />
-      </material>
-    </visual>
-    <collision>
-      <origin
-        xyz="0 0 0"
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
File: quadruped_description/xacros/transmission.xacro (robot description, xacro)
@@ -1,4 +1,4 @@
 <?xml version="1.0" encoding="utf-8"?>
-<robot name="quad_wheel" xmlns:xacro="http://www.ros.org/wiki/xacro">
+<robot name="quadruped" xmlns:xacro="http://www.ros.org/wiki/xacro">
     <xacro:macro name="leg_transmission" params="name">
         <transmission name="trans_${name}1">
